Commit message: joint type changed

File: robotis_description/robots/robotis_op3.urdf (robot description, URDF)
Before this commit: robot robotis_op3, 13 links, 12 joints
Joints:
- joint l_ank_pitch: limit effort=1000 velocity=100 -> lower=-2.199 upper=2.199 effort=1000 velocity=100; type continuous -> revolute
- joint l_ank_roll: limit effort=1000 velocity=100 -> lower=-2.199 upper=2.199 effort=1000 velocity=100; type continuous -> revolute
- joint l_hip_pitch: limit effort=1000 velocity=100 -> lower=-2.199 upper=2.199 effort=1000 velocity=100; type continuous -> revolute
- joint l_hip_roll: limit effort=1000 velocity=100 -> lower=-2.199 upper=2.199 effort=1000 velocity=100; type continuous -> revolute
- joint l_hip_yaw: limit effort=1000 velocity=100 -> lower=-2.199 upper=2.199 effort=1000 velocity=100; type continuous -> revolute
- joint l_knee: limit effort=1000 velocity=100 -> lower=-2.199 upper=2.199 effort=1000 velocity=100; type continuous -> revolute
- joint r_ank_pitch: limit effort=1000 velocity=100 -> lower=-2.199 upper=2.199 effort=1000 velocity=100; type continuous -> revolute
- joint r_ank_roll: limit effort=1000 velocity=100 -> lower=-2.199 upper=2.199 effort=1000 velocity=100; type continuous -> revolute
- joint r_hip_pitch: limit effort=1000 velocity=100 -> lower=-2.199 upper=2.199 effort=1000 velocity=100; type continuous -> revolute
- joint r_hip_roll: limit effort=1000 velocity=100 -> lower=-2.199 upper=2.199 effort=1000 velocity=100; type continuous -> revolute
- joint r_hip_yaw: limit effort=1000 velocity=100 -> lower=-2.199 upper=2.199 effort=1000 velocity=100; type continuous -> revolute
- joint r_knee: limit effort=1000 velocity=100 -> lower=-2.199 upper=2.199 effort=1000 velocity=100; type continuous -> revolute

Commit message: model update

File: robotis_description/robots/robotis_op3.urdf (robot description, URDF)
Before this commit: robot robotis_op3, 13 links, 12 joints
Joints:
- joint l_ank_pitch: limit lower=-2.199 upper=2.199 effort=1000 velocity=100 -> lower=-2.199 upper=2.199 effort=10 velocity=5
- joint l_ank_roll: limit lower=-2.199 upper=2.199 effort=1000 velocity=100 -> lower=-2.199 upper=2.199 effort=10 velocity=5
- joint l_hip_pitch: limit lower=-2.199 upper=2.199 effort=1000 velocity=100 -> lower=-2.199 upper=2.199 effort=10 velocity=5
- joint l_hip_roll: limit lower=-2.199 upper=2.199 effort=1000 velocity=100 -> lower=-2.199 upper=2.199 effort=10 velocity=5
- joint l_hip_yaw: limit lower=-2.199 upper=2.199 effort=1000 velocity=100 -> lower=-2.199 upper=2.199 effort=10 velocity=5
- joint l_knee: limit lower=-2.199 upper=2.199 effort=1000 velocity=100 -> lower=-2.199 upper=2.199 effort=10 velocity=5
- joint r_ank_pitch: limit lower=-2.199 upper=2.199 effort=1000 velocity=100 -> lower=-2.199 upper=2.199 effort=10 velocity=5
- joint r_ank_roll: limit lower=-2.199 upper=2.199 effort=1000 velocity=100 -> lower=-2.199 upper=2.199 effort=10 velocity=5
- joint r_hip_pitch: limit lower=-2.199 upper=2.199 effort=1000 velocity=100 -> lower=-2.199 upper=2.199 effort=10 velocity=5
- joint r_hip_roll: limit lower=-2.199 upper=2.199 effort=1000 velocity=100 -> lower=-2.199 upper=2.199 effort=10 velocity=5
- joint r_hip_yaw: limit lower=-2.199 upper=2.199 effort=1000 velocity=100 -> lower=-2.199 upper=2.199 effort=10 velocity=5
- joint r_knee: limit lower=-2.199 upper=2.199 effort=1000 velocity=100 -> lower=-2.199 upper=2.199 effort=10 velocity=5

Commit message: model update

File: robotis_description/robots/robotis_op3.urdf (robot description, URDF)
Before this commit: robot robotis_op3, 13 links, 12 joints
Links:
- added link imu_link
- added link l_foot_link, mass 0.05753; collision mesh filename=package://robotis_description/stl/ll6-2.stl scale=0.001 0.001 0.001; visual mesh filename=package://robotis_description/stl/ll6-2.stl scale=0.001 0.001 0.001
- added link l_leg_ft_link
- added link r_foot_link, mass 0.05753; collision mesh filename=package://robotis_description/stl/rl6-2.stl scale=0.001 0.001 0.001; visual mesh filename=package://robotis_description/stl/rl6-2.stl scale=0.001 0.001 0.001
- added link r_leg_ft_link
- link l_ank_roll_link: mass 0.06934 -> 0.01181
- link r_ank_roll_link: mass 0.06934 -> 0.01181; geometry collision mesh filename=package://robotis_description/stl/rl6-1.stl scale=0.001 0.001 0.001; visual mesh filename=package://robotis_description/stl/rl6-1.stl scale=0.001 0.001 0.001
Joints:
- added joint imu: type fixed, parent body_link, child imu_link, origin xyz=0.0 0.0 0.0 rpy=0 0 0
- added joint l_leg_ft: type revolute, parent l_ank_roll_link, child l_leg_ft_link, origin xyz=0.0241 0.0 -0.0285 rpy=0 0 0, limit lower=0 upper=0 effort=1000 velocity=6.5
- added joint l_leg_ft_fixed: type fixed, parent l_leg_ft_link, child l_foot_link
- added joint r_leg_ft: type revolute, parent r_ank_roll_link, child r_leg_ft_link, origin xyz=0.0241 0.0 -0.0285 rpy=0 0 0, limit lower=0 upper=0 effort=1000 velocity=6.5
- added joint r_leg_ft_fixed: type fixed, parent r_leg_ft_link, child r_foot_link
- joint l_ank_pitch: limit lower=-2.199 upper=2.199 effort=10 velocity=5 -> lower=-2.199 upper=2.199 effort=1000 velocity=100
- joint l_ank_roll: limit lower=-2.199 upper=2.199 effort=10 velocity=5 -> lower=-2.199 upper=2.199 effort=1000 velocity=100
- joint l_hip_pitch: limit lower=-2.199 upper=2.199 effort=10 velocity=5 -> lower=-2.199 upper=2.199 effort=1000 velocity=100
- joint l_hip_roll: limit lower=-2.199 upper=2.199 effort=10 velocity=5 -> lower=-2.199 upper=2.199 effort=1000 velocity=100
- joint l_hip_yaw: limit lower=-2.199 upper=2.199 effort=10 velocity=5 -> lower=-2.199 upper=2.199 effort=1000 velocity=100
- joint l_knee: limit lower=-2.199 upper=2.199 effort=10 velocity=5 -> lower=-2.199 upper=2.199 effort=1000 velocity=100
- joint r_ank_pitch: limit lower=-2.199 upper=2.199 effort=10 velocity=5 -> lower=-2.199 upper=2.199 effort=1000 velocity=100
- joint r_ank_roll: limit lower=-2.199 upper=2.199 effort=10 velocity=5 -> lower=-2.199 upper=2.199 effort=1000 velocity=100
- joint r_hip_pitch: limit lower=-2.199 upper=2.199 effort=10 velocity=5 -> lower=-2.199 upper=2.199 effort=1000 velocity=100
- joint r_hip_roll: limit lower=-2.199 upper=2.199 effort=10 velocity=5 -> lower=-2.199 upper=2.199 effort=1000 velocity=100
- joint r_hip_yaw: limit lower=-2.199 upper=2.199 effort=10 velocity=5 -> lower=-2.199 upper=2.199 effort=1000 velocity=100
- joint r_knee: limit lower=-2.199 upper=2.199 effort=10 velocity=5 -> lower=-2.199 upper=2.199 effort=1000 velocity=100

Commit message: model sensor added

File: robotis_description/robots/robotis_op3.urdf (robot description, URDF)
Before this commit: robot robotis_op3, 18 links, 17 joints
Links:
- link l_foot_link: geometry collision box size=0.13 0.0825 0.01; visual mesh filename=package://robotis_description/stl/ll6-2.stl scale=0.001 0.001 0.001
- link r_foot_link: geometry collision box size=0.13 0.0825 0.01; visual mesh filename=package://robotis_description/stl/rl6-2.stl scale=0.001 0.001 0.001

Commit message: package added

File: robotis_description/robots/robotis_op3.urdf (robot description, URDF)
Before this commit: robot robotis_op3, 18 links, 17 joints
Links:
- link l_foot_link: geometry collision box size=0.13 0.0825 0.005; visual mesh filename=package://robotis_description/stl/ll6-2.stl scale=0.001 0.001 0.001
- link r_foot_link: geometry collision box size=0.13 0.0825 0.005; visual mesh filename=package://robotis_description/stl/rl6-2.stl scale=0.001 0.001 0.001
